File: pcb/EVQWGD001_extension/EVQWGD001_extension.kicad_sch (KiCad schematic)
At the start: 6 parts, among them J1 Conn_01x01_MountingPin, J2 Conn_01x01_MountingPin, J3 Conn_01x01_MountingPin, J4 Conn_01x01_MountingPin, J5 Conn_01x01_MountingPin, SW1 RotaryEncoder_Switch

Commit message: add fp and symbol
Parts:
- J1, J2, J3, J4, J5: footprint Connector_PinSocket_2.54mm:PinSocket_1x01_P2.54mm_Vertical -> roBa:PinSocket_1x01_P2.54mm_Vertical
- SW1: footprint EVQWGD001:EVQWGD001 -> roBa:EVQWGD001
Changed lines of the file:
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@@
 			)
 		)
-		(property "Footprint" "EVQWGD001:EVQWGD001"
+		(property "Footprint" "roBa:EVQWGD001"
 			(at 140.97 96.266 0)
 			(effects
@@
 			)
 		)
-		(property "Footprint" "Connector_PinSocket_2.54mm:PinSocket_1x01_P2.54mm_Vertical"
+		(property "Footprint" "roBa:PinSocket_1x01_P2.54mm_Vertical"
 			(at 166.37 72.39 0)
 			(effects
@@
 			)
 		)
-		(property "Footprint" "Connector_PinSocket_2.54mm:PinSocket_1x01_P2.54mm_Vertical"
+		(property "Footprint" "roBa:PinSocket_1x01_P2.54mm_Vertical"
 			(at 179.07 72.39 0)
 			(effects
@@
 			)
 		)
-		(property "Footprint" "Connector_PinSocket_2.54mm:PinSocket_1x01_P2.54mm_Vertical"
+		(property "Footprint" "roBa:PinSocket_1x01_P2.54mm_Vertical"
 			(at 129.54 72.39 0)
 			(effects
@@
 			)
 		)
-		(property "Footprint" "Connector_PinSocket_2.54mm:PinSocket_1x01_P2.54mm_Vertical"
+		(property "Footprint" "roBa:PinSocket_1x01_P2.54mm_Vertical"
 			(at 118.11 72.39 0)
 			(effects
@@
 			)
 		)
-		(property "Footprint" "Connector_PinSocket_2.54mm:PinSocket_1x01_P2.54mm_Vertical"
+		(property "Footprint" "roBa:PinSocket_1x01_P2.54mm_Vertical"
 			(at 107.95 72.39 0)
 			(effects
