File: pcb/pmw3610_breakout_for_roBa/pmw3610_breakout_for_roBa.kicad_pcb (KiCad board)
At the start: 2 copper layers, 22 x 23.5 mm, 13 parts, among them J1 Conn_01x08, U1 MCP1700x-180xxTT, U2 PMW3610

Commit message: add fp and symbol
Parts:
- C1, C2, C3, C4, C5, C6, C7, C8: footprint Capacitor_SMD:C_0603_1608Metric -> roBa:C_0603_1608Metric
- C9: value 3.3u/16V -> 3.3u/25V; footprint Capacitor_SMD:C_0603_1608Metric -> roBa:C_0603_1608Metric
- J1: footprint myfootprintLibrary:pmw3610_connector -> roBa:pmw3610_connector_b
- R1: footprint Resistor_SMD:R_0603_1608Metric -> roBa:R_0603_1608Metric
- U1: value MCP1700x-180xxTT -> MCP1700T-1802E/TT; footprint Package_TO_SOT_SMD:SOT-23 -> roBa:SOT-23
- U2: footprint pmw3610_breakout:PMW3610DM-SUDU 16Pin -> roBa:PMW3610DM-SUDU 16Pin
Connections:
- net MOTION_2 renamed MOTION
- net NCS_2 renamed NCS
- net SCLK_2 renamed SCLK
- net SDIO_2 renamed SDIO
- J1 pad 5: unconnected-(J1-Pin_5-Pad5) -> (no net)
