File: pcb/pmw3610_breakout_for_roBa/pmw3610_breakout_for_roBa.kicad_sch (KiCad schematic)
At the start: 13 parts, among them J1 Conn_01x08, U1 MCP1700T-1802E/TT, U2 PMW3610

Commit message: add fp and symbol
Parts:
- C1, C2, C3, C4, C5, C6, C7, C8, C9: footprint Capacitor_SMD:C_0603_1608Metric -> roBa:C_0603_1608Metric
- J1: footprint myfootprintLibrary:pmw3610_connector -> roBa:pmw3610_connector_b
- R1: footprint Resistor_SMD:R_0603_1608Metric -> roBa:R_0603_1608Metric
- U1: footprint Package_TO_SOT_SMD:SOT-23 -> roBa:SOT-23
- U2: footprint PMW3610DM-SUDU 16Pin -> roBa:PMW3610DM-SUDU 16Pin
Changed lines of the file:
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@@
 			)
 		)
-		(property "Footprint" "PMW3610DM-SUDU 16Pin"
+		(property "Footprint" "roBa:PMW3610DM-SUDU 16Pin"
 			(at 142.24 86.36 0)
 			(effects
@@
 			)
 		)
-		(property "Footprint" "myfootprintLibrary:pmw3610_connector"
+		(property "Footprint" "roBa:pmw3610_connector_b"
 			(at 232.41 96.52 0)
 			(effects
@@
 			)
 		)
-		(property "Footprint" "Capacitor_SMD:C_0603_1608Metric"
+		(property "Footprint" "roBa:C_0603_1608Metric"
 			(at 80.01 96.52 0)
 			(effects
@@
 			)
 		)
-		(property "Footprint" "Package_TO_SOT_SMD:SOT-23"
+		(property "Footprint" "roBa:SOT-23"
 			(at 68.58 88.265 0)
 			(effects
@@
 			)
 		)
-		(property "Footprint" "Capacitor_SMD:C_0603_1608Metric"
+		(property "Footprint" "roBa:C_0603_1608Metric"
 			(at 109.22 105.41 0)
 			(effects
@@
 			)
 		)
-		(property "Footprint" "Capacitor_SMD:C_0603_1608Metric"
+		(property "Footprint" "roBa:C_0603_1608Metric"
 			(at 181.61 95.25 0)
 			(effects
@@
 			)
 		)
-		(property "Footprint" "Capacitor_SMD:C_0603_1608Metric"
+		(property "Footprint" "roBa:C_0603_1608Metric"
 			(at 165.1 85.09 0)
 			(effects
@@
 			)
 		)
-		(property "Footprint" "Capacitor_SMD:C_0603_1608Metric"
+		(property "Footprint" "roBa:C_0603_1608Metric"
 			(at 165.1 99.06 0)
 			(effects
@@
 			)
 		)
-		(property "Footprint" "Capacitor_SMD:C_0603_1608Metric"
+		(property "Footprint" "roBa:C_0603_1608Metric"
 			(at 57.15 96.52 0)
 			(effects
@@
 			)
 		)
-		(property "Footprint" "Resistor_SMD:R_0603_1608Metric"
+		(property "Footprint" "roBa:R_0603_1608Metric"
 			(at 114.808 115.824 90)
 			(effects
@@
 			)
 		)
-		(property "Footprint" "Capacitor_SMD:C_0603_1608Metric"
+		(property "Footprint" "roBa:C_0603_1608Metric"
 			(at 180.34 111.76 0)
 			(effects
@@
 			)
 		)
-		(property "Footprint" "Capacitor_SMD:C_0603_1608Metric"
+		(property "Footprint" "roBa:C_0603_1608Metric"
 			(at 189.23 95.25 0)
 			(effects
@@
 			)
 		)
-		(property "Footprint" "Capacitor_SMD:C_0603_1608Metric"
+		(property "Footprint" "roBa:C_0603_1608Metric"
 			(at 172.72 111.76 0)
 			(effects
