File: pcb/roBa_L/roba_L.kicad_sch (KiCad schematic)
At the start: 56 parts, among them J1 Conn_01x01-Connector_Generic, J2 Conn_01x01-Connector_Generic, J3 Conn_01x01-Connector_Generic, J4 Conn_01x01-Connector_Generic, J5 Conn_01x01-Connector_Generic, J6 Conn_01x01-Connector_Generic, J7 Conn_01x01-Connector_Generic, SW1 SW_PUSH, SW10 SW_PUSH, SW11 SW_PUSH, SW12 SW_PUSH, SW13 SW_PUSH, SW14 SW_PUSH, SW15 SW_PUSH, SW16 SW_PUSH, SW17 SW_PUSH, SW18 SW_PUSH, SW19 SW_PUSH, SW2 SW_PUSH, SW20 SW_PUSH, SW21 RotaryEncoder_Switch, SW22 SW_PUSH, SW23 SW_PUSH, SW24 SW_SPDT, SW3 SW_PUSH, SW4 SW_PUSH, SW5 SW_PUSH, SW6 SW_PUSH, SW7 SW_PUSH, SW8 SW_PUSH, SW9 SW_PUSH

Commit message: add fp and symbol
Parts:
- B1: footprint note96e:JST_PH_S2B-PH-K_custom -> roBa:JST_PH_S2B-PH-K_custom
- D1, D10, D11, D12, D13, D14, D15, D16, D17, D18, D19, D2, D20, D21, D22, D23, D3, D4, D5, D6, D7, D8, D9: footprint note96e:Diode_SMD -> roBa:Diode_SMD
- SW1, SW10, SW11, SW12, SW13, SW14, SW15, SW17, SW18, SW19, SW2, SW22, SW3, SW4, SW5, SW6, SW7, SW8, SW9: footprint myfootprintLibrary:SW_MX -> roBa:SW_MX
- SW16, SW20, SW23: footprint myfootprintLibrary:SW_MX -> roBa:SW_MX_Choc
- SW21: footprint myfootprintLibrary:SW_MX_EC12 -> roBa:SW_MX_EC12
- SW24: footprint note96e:TGSW_MSK-12D19 -> roBa:TGSW_MSK-12D19
- U1: footprint myfootprintLibrary:XIAO_nRF52840_wBAT_wNFC -> roBa:XIAO_nRF52840_wBAT_wNFC
Changed lines of the file:
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@@
 			)
 		)
-		(property "Footprint" "note96e:Diode_SMD"
+		(property "Footprint" "roBa:Diode_SMD"
 			(at 149.86 72.39 0)
 			(effects
@@
 			)
 		)
-		(property "Footprint" "note96e:Diode_SMD"
+		(property "Footprint" "roBa:Diode_SMD"
 			(at 168.91 53.34 0)
 			(effects
@@
 			)
 		)
-		(property "Footprint" "note96e:Diode_SMD"
+		(property "Footprint" "roBa:Diode_SMD"
 			(at 226.06 91.44 0)
 			(effects
@@
 			)
 		)
-		(property "Footprint" "note96e:Diode_SMD"
+		(property "Footprint" "roBa:Diode_SMD"
 			(at 149.86 109.22 0)
 			(effects
@@
 			)
 		)
-		(property "Footprint" "note96e:Diode_SMD"
+		(property "Footprint" "roBa:Diode_SMD"
 			(at 168.91 72.39 0)
 			(effects
@@
 			)
 		)
-		(property "Footprint" "note96e:Diode_SMD"
+		(property "Footprint" "roBa:Diode_SMD"
 			(at 226.06 72.39 0)
 			(effects
@@
 			)
 		)
-		(property "Footprint" "myfootprintLibrary:SW_MX_EC12"
+		(property "Footprint" "roBa:SW_MX_EC12"
 			(at 248.92 124.206 0)
 			(effects
@@
 			)
 		)
-		(property "Footprint" "myfootprintLibrary:SW_MX"
+		(property "Footprint" "roBa:SW_MX"
 			(at 173.99 49.53 0)
 			(effects
@@
 			)
 		)
-		(property "Footprint" "myfootprintLibrary:XIAO_nRF52840_wBAT_wNFC"
+		(property "Footprint" "roBa:XIAO_nRF52840_wBAT_wNFC"
 			(at 41.91 50.8 0)
 			(effects
@@
 			)
 		)
-		(property "Footprint" "myfootprintLibrary:SW_MX"
+		(property "Footprint" "roBa:SW_MX"
 			(at 154.94 105.41 0)
 			(effects
@@
 			)
 		)
-		(property "Footprint" "note96e:Diode_SMD"
+		(property "Footprint" "roBa:Diode_SMD"
 			(at 149.86 53.34 0)
 			(effects
@@
 			)
 		)
-		(property "Footprint" "myfootprintLibrary:SW_MX"
+		(property "Footprint" "roBa:SW_MX"
 			(at 193.04 49.53 0)
 			(effects
@@
 			)
 		)
-		(property "Footprint" "note96e:Diode_SMD"
+		(property "Footprint" "roBa:Diode_SMD"
 			(at 130.81 91.44 0)
 			(effects
@@
 			)
 		)
-		(property "Footprint" "myfootprintLibrary:SW_MX"
+		(property "Footprint" "roBa:SW_MX"
 			(at 135.89 68.58 0)
 			(effects
@@
 			)
 		)
-		(property "Footprint" "myfootprintLibrary:SW_MX"
+		(property "Footprint" "roBa:SW_MX"
 			(at 173.99 87.63 0)
 			(effects
@@
 			)
 		)
-		(property "Footprint" "myfootprintLibrary:SW_MX"
+		(property "Footprint" "roBa:SW_MX"
 			(at 154.94 49.53 0)
 			(effects
@@
 			)
 		)
-		(property "Footprint" "myfootprintLibrary:SW_MX"
+		(property "Footprint" "roBa:SW_MX"
 			(at 154.94 87.63 0)
 			(effects
@@
 			)
 		)
-		(property "Footprint" "myfootprintLibrary:SW_MX"
+		(property "Footprint" "roBa:SW_MX"
 			(at 173.99 104.14 0)
 			(effects
@@
 			)
 		)
-		(property "Footprint" "note96e:Diode_SMD"
+		(property "Footprint" "roBa:Diode_SMD"
 			(at 207.01 109.22 0)
 			(effects
@@
 			)
 		)
-		(property "Footprint" "note96e:Diode_SMD"
+		(property "Footprint" "roBa:Diode_SMD"
 			(at 130.81 53.34 0)
 			(effects
@@
 			)
 		)
-		(property "Footprint" "myfootprintLibrary:SW_MX"
+		(property "Footprint" "roBa:SW_MX_Choc"
 			(at 193.04 105.41 0)
 			(effects
@@
 			)
 		)
-		(property "Footprint" "note96e:Diode_SMD"
+		(property "Footprint" "roBa:Diode_SMD"
 			(at 226.06 109.22 0)
 			(effects
@@
 			)
 		)
-		(property "Footprint" "note96e:Diode_SMD"
+		(property "Footprint" "roBa:Diode_SMD"
 			(at 187.96 72.39 0)
 			(effects
@@
 			)
 		)
-		(property "Footprint" "myfootprintLibrary:SW_MX"
+		(property "Footprint" "roBa:SW_MX"
 			(at 193.04 68.58 0)
 			(effects
@@
 			)
 		)
-		(property "Footprint" "note96e:Diode_SMD"
+		(property "Footprint" "roBa:Diode_SMD"
 			(at 207.01 91.44 0)
 			(effects
@@
 			)
 		)
-		(property "Footprint" "myfootprintLibrary:SW_MX"
+		(property "Footprint" "roBa:SW_MX_Choc"
 			(at 212.09 105.41 0)
 			(effects
@@
 			)
 		)
-		(property "Footprint" "note96e:Diode_SMD"
+		(property "Footprint" "roBa:Diode_SMD"
 			(at 187.96 91.44 0)
 			(effects
@@
 			)
 		)
-		(property "Footprint" "myfootprintLibrary:SW_MX"
+		(property "Footprint" "roBa:SW_MX"
 			(at 193.04 87.63 0)
 			(effects
@@
 			)
 		)
-		(property "Footprint" "myfootprintLibrary:SW_MX"
+		(property "Footprint" "roBa:SW_MX"
 			(at 212.09 49.53 0)
 			(effects
@@
 			)
 		)
-		(property "Footprint" "myfootprintLibrary:SW_MX"
+		(property "Footprint" "roBa:SW_MX"
 			(at 173.99 68.58 0)
 			(effects
@@
 			)
 		)
-		(property "Footprint" "note96e:Diode_SMD"
+		(property "Footprint" "roBa:Diode_SMD"
 			(at 168.91 109.22 0)
 			(effects
@@
 			)
 		)
-		(property "Footprint" "note96e:Diode_SMD"
+		(property "Footprint" "roBa:Diode_SMD"
 			(at 130.81 72.39 0)
 			(effects
@@
 			)
 		)
-		(property "Footprint" "note96e:Diode_SMD"
+		(property "Footprint" "roBa:Diode_SMD"
 			(at 207.01 72.39 0)
 			(effects
@@
 			)
 		)
-		(property "Footprint" "myfootprintLibrary:SW_MX"
+		(property "Footprint" "roBa:SW_MX"
 			(at 231.14 87.63 0)
 			(effects
@@
 			)
 		)
-		(property "Footprint" "note96e:Diode_SMD"
+		(property "Footprint" "roBa:Diode_SMD"
 			(at 149.86 91.44 0)
 			(effects
@@
 			)
 		)
-		(property "Footprint" "myfootprintLibrary:SW_MX"
+		(property "Footprint" "roBa:SW_MX"
 			(at 212.09 68.58 0)
 			(effects
@@
 			)
 		)
-		(property "Footprint" "myfootprintLibrary:SW_MX"
+		(property "Footprint" "roBa:SW_MX_Choc"
 			(at 231.14 105.41 0)
 			(effects
@@
 			)
 		)
-		(property "Footprint" "myfootprintLibrary:SW_MX"
+		(property "Footprint" "roBa:SW_MX"
 			(at 135.89 105.41 0)
 			(effects
@@
 			)
 		)
-		(property "Footprint" "myfootprintLibrary:SW_MX"
+		(property "Footprint" "roBa:SW_MX"
 			(at 212.09 87.63 0)
 			(effects
@@
 			)
 		)
-		(property "Footprint" "note96e:Diode_SMD"
+		(property "Footprint" "roBa:Diode_SMD"
 			(at 187.96 53.34 0)
 			(effects
@@
 			)
 		)
-		(property "Footprint" "myfootprintLibrary:SW_MX"
+		(property "Footprint" "roBa:SW_MX"
 			(at 154.94 68.58 0)
 			(effects
@@
 			)
 		)
-		(property "Footprint" "note96e:JST_PH_S2B-PH-K_custom"
+		(property "Footprint" "roBa:JST_PH_S2B-PH-K_custom"
 			(at 68.834 160.02 90)
 			(effects
@@
 			)
 		)
-		(property "Footprint" "note96e:TGSW_MSK-12D19"
+		(property "Footprint" "roBa:TGSW_MSK-12D19"
 			(at 55.88 160.02 0)
 			(effects
@@
 			)
 		)
-		(property "Footprint" "note96e:Diode_SMD"
+		(property "Footprint" "roBa:Diode_SMD"
 			(at 130.81 109.22 0)
 			(effects
@@
 			)
 		)
-		(property "Footprint" "note96e:Diode_SMD"
+		(property "Footprint" "roBa:Diode_SMD"
 			(at 187.96 109.22 0)
 			(effects
@@
 			)
 		)
-		(property "Footprint" "myfootprintLibrary:SW_MX"
+		(property "Footprint" "roBa:SW_MX"
 			(at 135.89 87.63 0)
 			(effects
@@
 			)
 		)
-		(property "Footprint" "myfootprintLibrary:SW_MX"
+		(property "Footprint" "roBa:SW_MX"
 			(at 135.89 49.53 0)
 			(effects
@@
 			)
 		)
-		(property "Footprint" "note96e:Diode_SMD"
+		(property "Footprint" "roBa:Diode_SMD"
 			(at 207.01 53.34 0)
 			(effects
@@
 			)
 		)
-		(property "Footprint" "note96e:Diode_SMD"
+		(property "Footprint" "roBa:Diode_SMD"
 			(at 168.91 91.44 0)
 			(effects
