File: pcb/roBa_R/roba_R.kicad_sch (KiCad schematic)
At the start: 50 parts, among them J2 Conn_01x01-Connector_Generic, J3 Conn_01x01-Connector_Generic, J4 Conn_01x01-Connector_Generic, J5 Conn_01x01-Connector_Generic, J6 Conn_01x01-Connector_Generic, J7 Conn_01x01-Connector_Generic, SW1 SW_PUSH, SW10 SW_PUSH, SW11 SW_PUSH, SW12 SW_PUSH, SW13 SW_PUSH, SW14 SW_PUSH, SW15 SW_PUSH, SW16 SW_PUSH, SW17 SW_PUSH, SW18 SW_PUSH, SW19 SW_PUSH, SW2 SW_PUSH, SW20 SW_PUSH, SW21 SW_SPDT, SW3 SW_PUSH, SW4 SW_PUSH, SW5 SW_PUSH, SW6 SW_PUSH, SW7 SW_PUSH, SW8 SW_PUSH, SW9 SW_PUSH

Commit message: add fp and symbol
Parts:
- BT1: footprint note96e:JST_PH_S2B-PH-K_custom -> roBa:JST_PH_S2B-PH-K_custom
- D1, D10, D11, D12, D13, D14, D15, D16, D17, D18, D19, D2, D20, D3, D4, D5, D6, D7, D8, D9: footprint note96e:Diode_SMD -> roBa:Diode_SMD
- J1: footprint myfootprintLibrary:pmw3610_connector -> roBa:pmw3610_connector
- SW1, SW10, SW11, SW13, SW14, SW15, SW17, SW18, SW19, SW2, SW20, SW3, SW4, SW5, SW6, SW7, SW8, SW9: footprint myfootprintLibrary:SW_MX -> roBa:SW_MX
- SW12, SW16: footprint myfootprintLibrary:SW_MX_Choc -> roBa:SW_MX_Choc
- SW21: footprint note96e:TGSW_MSK-12D19 -> roBa:TGSW_MSK-12D19
- U1: footprint myfootprintLibrary:XIAO_nRF52840_wBAT_wNFC -> roBa:XIAO_nRF52840_wBAT_wNFC
